File: kicad/h_bridge.kicad_sch (KiCad schematic)
At the start: 23 parts, among them U2 LTV-817S

Commit message: вариант с микросхемами a4950
Parts:
- C2: renamed from C1; value (none) -> C; footprint (none) -> Capacitor_THT:C_Radial_D10.0mm_H16.0mm_P5.00mm
- D5: renamed from D1; value (none) -> SS14; footprint (none) -> digikey-footprints:DO-214AC
- D6: renamed from D2; value (none) -> SS14; footprint (none) -> digikey-footprints:DO-214AC
- D7: renamed from D3; value (none) -> SS14; footprint (none) -> digikey-footprints:DO-214AC
- D8: renamed from D4; value (none) -> SS14; footprint (none) -> digikey-footprints:DO-214AC
- Q10: renamed from Q5; value (none) -> BC807-40_215; footprint (none) -> digikey-footprints:SOT-23-3
- Q11: renamed from Q6; value (none) -> BC817-40_215; footprint (none) -> digikey-footprints:SOT-23-3
- Q12: renamed from Q7; value (none) -> BC807-40_215; footprint (none) -> digikey-footprints:SOT-23-3
- Q13: renamed from Q8; value (none) -> BC817-40_215; footprint (none) -> digikey-footprints:SOT-23-3
- Q4: renamed from Q1; value (none) -> BC817-40_215; footprint (none) -> digikey-footprints:SOT-23-3
- R1: renamed from R3; value (none) -> 50; footprint (none) -> Resistor_SMD:R_0805_2012Metric
- R12: renamed from R5; value (none) -> 1.2k; footprint (none) -> Resistor_SMD:R_1206_3216Metric
- R30: renamed from R10; value (none) -> 100; footprint (none) -> Resistor_SMD:R_0805_2012Metric
- R31: renamed from R11; value (none) -> 1k; footprint (none) -> Resistor_SMD:R_0805_2012Metric
- R33: renamed from R13; value (none) -> 1k; footprint (none) -> Resistor_SMD:R_0805_2012Metric
- R34: renamed from R14; value (none) -> 1k; footprint (none) -> Resistor_SMD:R_0805_2012Metric
- R36: renamed from R16; value (none) -> 1k; footprint (none) -> Resistor_SMD:R_0805_2012Metric
- R6: renamed from R1; value (none) -> 1.2k; footprint (none) -> Resistor_SMD:R_1206_3216Metric
- R7: renamed from R2; value (none) -> 1.2k; footprint (none) -> Resistor_SMD:R_1206_3216Metric
- R8: renamed from R3; value (none) -> 1.5k; footprint (none) -> Resistor_SMD:R_0805_2012Metric
- R9: renamed from R4; value (none) -> 1.2k; footprint (none) -> Resistor_SMD:R_1206_3216Metric
- U3: renamed from U5; value (none) -> LTV-817S; footprint (none) -> Package_DIP:SMDIP-4_W9.53mm
- renumbered U2 to U4
