File: kicad/smart_window.kicad_sch (KiCad schematic)
At the start: 17 parts, among them J1 PROG, J7 I2C

Commit message: вариант с микросхемами a4950
Parts:
- removed J14, J2: (no value), Connector_JST:JST_XH_B2B-XH-A_1x02_P2.50mm_Vertical, symbol Connector:Conn_01x02_Male
- added C1, C2: (no value), symbol Device:C
- added C3, C5: 100µF, Capacitor_SMD:CP_Elec_10x10.5, symbol Device:C
- added C4, C6: 0.22µF, Capacitor_SMD:C_1206_3216Metric, symbol Device:C
- added R1, R2, R3: (no value), symbol Device:R
- added U3: (no value), symbol Driver_Motor:A4950E
- added U4, U5: A4950E, Package_SO:SOIC-8-1EP_3.9x4.9mm_P1.27mm_EP2.41x3.3mm, symbol Driver_Motor:A4950E
- J10: value (none) -> LS2; footprint (none) -> Connector_JST:JST_XH_B2B-XH-A_1x02_P2.50mm_Vertical
- J12: value (none) -> LS3; footprint (none) -> Connector_JST:JST_XH_B2B-XH-A_1x02_P2.50mm_Vertical
- J13: value (none) -> Vmot1
- J3: value (none) -> DOOR1; footprint (none) -> Connector_JST:JST_XH_B2B-XH-A_1x02_P2.50mm_Vertical
- J4: value (none) -> MOT2; footprint (none) -> Connector_JST:JST_XH_B2B-XH-A_1x02_P2.50mm_Vertical
- J5: value (none) -> MOT1; footprint (none) -> Connector_JST:JST_XH_B2B-XH-A_1x02_P2.50mm_Vertical
- J6: value (none) -> MOT3; footprint (none) -> Connector_JST:JST_XH_B2B-XH-A_1x02_P2.50mm_Vertical
- J8: value (none) -> DOOR2; footprint (none) -> Connector_JST:JST_XH_B2B-XH-A_1x02_P2.50mm_Vertical
- J9: value (none) -> LS1; footprint (none) -> Connector_JST:JST_XH_B2B-XH-A_1x02_P2.50mm_Vertical
- R4: value (none) -> A9050; footprint (none) -> OptoDevice:R_LDR_5.0x4.1mm_P3mm_Vertical
- R5: value (none) -> 500; footprint (none) -> Resistor_SMD:R_0805_2012Metric
- U1: value (none) -> ESP-12F; footprint (none) -> RF_Module:ESP-12E
- U2: value (none) -> MP1584EN 3.3V
Connections:
- net 24V-1 is gone; now on net GND: J13.2 (Pin_2), U2.4 (Vin-)
- net +3V3: now also U3.4 (VREF), U4.4 (VREF), U5.4 (VREF)
- net DOOR1: now also U1.4 (GPIO16); no longer U1.5 (GPIO14)
- net DOOR2: now also U1.5 (GPIO14); no longer U1.6 (GPIO12)
- net GND: now also C1.1, C2.1, C3.1, C4.1, C5.1, C6.1, R1.1, R2.1, R3.1, U3.1 (GND), U3.9 (PAD), U4.1 (GND), U4.9 (PAD), U5.1 (GND), U5.9 (PAD)
- net M1_DIR: now also U1.10 (MISO), U3.2 (IN2); no longer U1.17 (GPIO2)
- net M1_EN: now also U1.6 (GPIO12), U3.3 (IN1); no longer U1.14 (SCLK)
- net M2_DIR: now also U4.2 (IN2)
- net M2_EN: now also U4.3 (IN1)
- net M3_DIR: now also U1.14 (SCLK), U5.2 (IN2); no longer U1.10 (MISO)
- net M3_EN: now also U1.17 (GPIO2), U5.3 (IN1); no longer U1.9 (CS0)
- net 24V+1 renamed 24V+
- net 24V+: now also C1.2, C2.2, C3.2, C4.2, C5.2, C6.2, U3.5 (VBB), U4.5 (VBB), U5.5 (VBB)
- net h_bridge1/ML: no longer names the net of J5.1 (Pin_1)
- net h_bridge1/ML: now also U3.6 (OUT1)
- net h_bridge1/MR: no longer names the net of J5.2 (Pin_2)
- net h_bridge1/MR: now also U3.8 (OUT2)
- net h_bridge2/ML: no longer names the net of J4.1 (Pin_1)
- net h_bridge2/ML: now also U4.6 (OUT1)
- net h_bridge2/MR: no longer names the net of J4.2 (Pin_2)
- net h_bridge2/MR: now also U4.8 (OUT2)
- net h_bridge3/ML: no longer names the net of J6.1 (Pin_1)
- net h_bridge3/ML: now also U5.6 (OUT1)
- net h_bridge3/MR: no longer names the net of J6.2 (Pin_2)
- net h_bridge3/MR: now also U5.8 (OUT2)
- new net: R3.2, U5.7 (LSS)
- new net: R1.2, U3.7 (LSS)
- new net: R2.2, U4.7 (LSS)
Other:
- removed sheet h_bridge1
- removed sheet h_bridge2
- removed sheet h_bridge3
- moved on the sheet: J10, J12, J13, J4, J5, J6, J9

Commit message: 2-сторонняя версия
Parts:
- added H1: (no value), symbol Mechanical:MountingHole
- added H2: MountingHole, MountingHole:MountingHole_3.2mm_M3, symbol Mechanical:MountingHole
- C1: value (none) -> 100µF; footprint (none) -> Capacitor_SMD:CP_Elec_10x10.5
- C2: value (none) -> 0.22µF; footprint (none) -> Capacitor_SMD:C_1206_3216Metric
- J1: value PROG -> (none); footprint Connector_JST:JST_XH_B4B-XH-A_1x04_P2.50mm_Vertical -> (none)
- J10: value LS2 -> (none); footprint Connector_JST:JST_XH_B2B-XH-A_1x02_P2.50mm_Vertical -> (none)
- J12: value LS3 -> (none); footprint Connector_JST:JST_XH_B2B-XH-A_1x02_P2.50mm_Vertical -> (none)
- J3: value DOOR1 -> (none); footprint Connector_JST:JST_XH_B2B-XH-A_1x02_P2.50mm_Vertical -> (none)
- J7: value I2C -> (none); footprint Connector_JST:JST_XH_B4B-XH-A_1x04_P2.50mm_Vertical -> (none)
- J8: value DOOR2 -> (none); footprint Connector_JST:JST_XH_B2B-XH-A_1x02_P2.50mm_Vertical -> (none)
- J9: value LS1 -> (none); footprint Connector_JST:JST_XH_B2B-XH-A_1x02_P2.50mm_Vertical -> (none)
- R1, R2, R3: value (none) -> 0.2; footprint (none) -> Resistor_SMD:R_1206_3216Metric
- U3: value (none) -> A4950E; footprint (none) -> Package_SO:SOIC-8-1EP_3.9x4.9mm_P1.27mm_EP2.41x3.3mm
